File: Duet-master/Duet0.8.5/_saved_Headers.sch (KiCad schematic (older format))
At the start: 19 parts, among them J10 GND V_IN, J11 GND V_IN, J12 E1 TEMP, J13 Probe, J14 Z MOTOR, J15 Y MOTOR, J16 X MOTOR, J17 E0 MOTOR, J18 E1 MOTOR, J6 EXPANSION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

Commit message: Module Library update
Lots of duplicate footprints
Parts:
- J10, J11: footprint (none) -> Melter_Connections:JUMPER
- J12: footprint (none) -> Melter_Connections:PIN_ARRAY_2X1
- J13: footprint (none) -> Melter_Connections:PIN_ARRAY_4x1
- J6: footprint (none) -> Melter_Connections:PIN_ARRAY_25X2
- J7: footprint (none) -> Melter_Connections:PIN_ARRAY_5x2
- J8: footprint (none) -> Melter_Connections:V_TERM_2-WAY_6.35mm
- J9: footprint (none) -> Melter_Connections:5VPSGND_PIN_ARRAY_3X1
Changed lines of the file:
@@
 F 0 "J13" H 7000 9450 50  0000 C CNN
 F 1 "Probe" V 7150 9200 50  0000 C CNN
-F 2 "" H 7000 9200 60  0001 C CNN
+F 2 "Melter_Connections:PIN_ARRAY_4x1" H 7000 9200 60  0001 C CNN
 F 3 "" H 7000 9200 60  0001 C CNN
 	1    7000 9200
@@
 F 0 "J10" H 7000 6600 40  0000 C CNN
 F 1 "GND  V_IN" V 7150 6750 40  0000 C CNN
-F 2 "" H 7000 6700 60  0001 C CNN
+F 2 "Melter_Connections:JUMPER" H 7000 6700 60  0001 C CNN
 F 3 "" H 7000 6700 60  0001 C CNN
 	1    7000 6700
@@
 F 0 "J9" V 6950 5750 50  0000 C CNN
 F 1 "5V_PS" V 7150 5750 40  0000 C CNN
-F 2 "" H 7000 5750 60  0001 C CNN
+F 2 "Melter_Connections:5VPSGND_PIN_ARRAY_3X1" H 7000 5750 60  0001 C CNN
 F 3 "" H 7000 5750 60  0001 C CNN
 	1    7000 5750
@@
 F 0 "J6" H 3950 1770 60  0000 C CNN
 F 1 "EXPANSION" H 3950 9370 60  0000 C CNN
-F 2 "" H 3950 5700 60  0001 C CNN
+F 2 "Melter_Connections:PIN_ARRAY_25X2" H 3950 5700 60  0001 C CNN
 F 3 "" H 3950 5700 60  0001 C CNN
 	1    3950 5700
@@
 F 0 "J8" H 7000 4600 40  0000 C CNN
 F 1 "POWER IN" V 7150 4750 40  0000 C CNN
-F 2 "" H 7000 4700 60  0001 C CNN
+F 2 "Melter_Connections:V_TERM_2-WAY_6.35mm" H 7000 4700 60  0001 C CNN
 F 3 "" H 7000 4700 60  0001 C CNN
 	1    7000 4700
@@
 F 0 "J12" H 7000 8050 40  0000 C CNN
 F 1 "E1 TEMP" V 7150 8200 40  0000 C CNN
-F 2 "" H 7000 8150 60  0001 C CNN
+F 2 "Melter_Connections:PIN_ARRAY_2X1" H 7000 8150 60  0001 C CNN
 F 3 "" H 7000 8150 60  0001 C CNN
 	1    7000 8150
@@
 F 0 "J7" H 5250 3050 50  0000 C CNN
 F 1 "PanelDUE" V 5400 2800 50  0000 C CNN
-F 2 "" H 5250 2800 60  0001 C CNN
+F 2 "Melter_Connections:PIN_ARRAY_5x2" H 5250 2800 60  0001 C CNN
 F 3 "" H 5250 2800 60  0001 C CNN
 	1    5250 2800
@@
 F 0 "J11" H 7000 6900 40  0000 C CNN
 F 1 "GND  V_IN" V 7150 7050 40  0000 C CNN
-F 2 "" H 7000 7000 60  0001 C CNN
+F 2 "Melter_Connections:JUMPER" H 7000 7000 60  0001 C CNN
 F 3 "" H 7000 7000 60  0001 C CNN
 	1    7000 7000
