File: Duet-master/Duet0.8.5/_saved_Processor.sch (KiCad schematic (older format))
At the start: 43 parts, among them J23 JTAG, J24 GND, U12 ATSAM3X8E, X2 CRYSTAL_4PIN

Commit message: PCB layout of components started
Experienced advice welcome.
Parts:
- C92: footprint (none) -> Melter_Connections:0mf01_Capacitor
- J23: footprint (none) -> Melter_Connections:PIN_ARRAY_5x2
- J24: footprint (none) -> Melter_Connections:GND_TP
- R103: footprint (none) -> Melter_Connections:6k8_R_0603
- U12: footprint LQFP100 -> Melter_Connections:LQFP144
Changed lines of the file:
@@
 F 0 "J24" H 10850 14450 60  0000 C CNN
 F 1 "GND" H 10550 14450 60  0000 C CNN
-F 2 "" H 10750 14200 60  0001 C CNN
+F 2 "Melter_Connections:GND_TP" H 10750 14200 60  0001 C CNN
 F 3 "" H 10750 14200 60  0001 C CNN
 	1    10750 14200
@@
 F 0 "U12" H 12050 9600 60  0000 C CNN
 F 1 "ATSAM3X8E" H 12050 9450 60  0000 C CNN
-F 2 "LQFP100" H 12050 9300 60  0000 C CNN
+F 2 "Melter_Connections:LQFP144" H 12050 9300 60  0000 C CNN
 F 3 "" H 12050 8950 60  0001 C CNN
 	1    12050 8950
@@
 F 0 "R103" V 9675 12958 50  0000 C CNN
 F 1 "6k8" V 9532 12962 50  0000 C CNN
-F 2 "" H 9600 12950 60  0001 C CNN
+F 2 "Melter_Connections:6k8_R_0603" H 9600 12950 60  0001 C CNN
 F 3 "" H 9600 12950 60  0001 C CNN
 	1    9600 12950
@@
 F 0 "C92" H 15575 12375 50  0000 L CNN
 F 1 "0u01" H 15550 12225 50  0000 L CNN
-F 2 "" H 15550 12300 60  0001 C CNN
+F 2 "Melter_Connections:0mf01_Capacitor" H 15550 12300 60  0001 C CNN
 F 3 "" H 15550 12300 60  0001 C CNN
 	1    15550 12300
@@
 F 0 "J23" H 8650 8150 50  0000 C CNN
 F 1 "JTAG" H 8650 8750 35  0000 C CNN
-F 2 "" H 8650 8450 60  0001 C CNN
+F 2 "Melter_Connections:PIN_ARRAY_5x2" H 8650 8450 60  0001 C CNN
 F 3 "" H 8650 8450 60  0001 C CNN
 	1    8650 8450
