File: Duet-master/Duet0.8.5/Htr_Fan.sch (KiCad schematic (older format))
At the start: 57 parts, among them J22 GND

Commit message: PCB layout of components started
Experienced advice welcome.
Parts:
- C62, C63, C68: footprint (none) -> Melter_Connections:10mf_capacitor
- C64, C65: footprint (none) -> Melter_Connections:0mf1_capacitor
- C66, C67: footprint (none) -> Melter_Connections:100mf_capacitor
- D18: footprint (none) -> Melter_Connections:BED_Diode_0603
- D19: footprint (none) -> Melter_Connections:E0_Diode_0603
- D20, D21, D22, D23, D24, D25: footprint (none) -> Melter_Connections:LED0_diode
- D26: footprint (none) -> Melter_Connections:FAN0_diode
- D27: footprint (none) -> Melter_Connections:FAN1_diode
- J22: footprint (none) -> Melter_Connections:GND_TP
- R100, R101, R79, R82, R83, R84, R85, R88, R89, R92, R93, R96, R97: footprint (none) -> Melter_Connections:4k7_R_0603
- R75, R76: footprint (none) -> Melter_Connections:100k_R_0603
- R77, R78: footprint (none) -> Melter_Connections:470R_R_0603
- R80, R81: footprint (none) -> Melter_Connections:220R_R_0603
- R86, R87, R90, R91, R94, R95, R98, R99: footprint (none) -> Melter_Connections:10k_R_0603
- TR10, TR11, TR12, TR13, TR6, TR7, TR8, TR9: footprint (none) -> Melter_Connections:PMV40UN2_SOT-23
- TR2, TR3: footprint (none) -> Melter_Connections:BSH105_SOT-23
- TR4, TR5: footprint (none) -> Melter_Connections:IPD036N04L_D-PAK
