File: Duet-master/Duet0.8.5/Stepper_Drv.sch (KiCad schematic (older format))
At the start: 112 parts, among them J1 X VREF, J2 Z VREF, J3 Y VREF, J4 E0 VREF, J5 E1 VREF, U1 A4982SLPTR, U2 A4982SLPTR, U3 A4982SLPTR, U4 A4982SLPTR, U5 A4982SLPTR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

Commit message: PCB layout of components started
Experienced advice welcome.
Parts:
- D1: footprint (none) -> Melter_Connections:1SS400T1G
- D2: footprint (none) -> Melter_Connections:E1STOP_diode
- D3: footprint (none) -> Melter_Connections:YSTOP_diode
- D4: footprint (none) -> Melter_Connections:ZSTOP_diode
- D5: footprint (none) -> Melter_Connections:E2STOP_diode
- D6: footprint (none) -> Melter_Connections:E0STOP_diode
- D7: footprint (none) -> Melter_Connections:XSTOP_diode
- J1, J2, J3, J4, J5: footprint (none) -> Melter_Connections:Vref
- R1, R13, R22, R3, R31: footprint (none) -> Melter_Connections:100k_R_0603
- R10, R17, R18, R19, R20, R28, R29, R7, R8, R9: footprint (none) -> Melter_Connections:0R1_R_1206
- R11: footprint 0603 -> Melter_Connections:100k_R_0603
- R12, R14, R2, R23, R30, R4: footprint (none) -> Melter_Connections:10k_R_0603
- R15, R16, R25, R5, R6: footprint (none) -> Melter_Connections:0R_R_0603
- R21, R24: footprint (none) -> Melter_Connections:4k7_R_0603
- R26: footprint (none) -> Melter_Connections:2k7_R_0603
- R27: footprint (none) -> Melter_Connections:2k15_R_0603
- R32, R33, R37, R38, R39: footprint (none) -> Melter_Connections:100R_R_0603
- R34, R35, R36, R40, R41, R42: footprint (none) -> Melter_Connections:680R_R_0603
- SJ1, SJ10, SJ2, SJ3, SJ4, SJ5, SJ6, SJ7, SJ8, SJ9: footprint (none) -> Melter_Connections:SJump
- U1, U2, U3, U4, U5: footprint (none) -> Melter_Connections:A4982SPLTR_TSSOP-24-thin_pads
- U6: footprint (none) -> Melter_Connections:MCP44X1_TSSOP-20
