File: Duet-master/Duet0.8.5/Duet0.85.kicad_pcb (KiCad board)
At the start: 4 copper layers, 286.6 x 277.8 mm, 318 parts, among them J1 X VREF, J10 GND V_IN, J11 GND V_IN, J12 E1 TEMP, J13 Probe, J19 USB, J2 Z VREF, J20 uSDHC, J21 ETHERNET, J22 GND, J23 JTAG, J24 GND, J3 Y VREF, J4 E0 VREF, J5 E1 VREF, J6 EXPANSION, J7 PanelDUE, J8 POWER IN, J9 5V_PS, P1 CONN_4, P2 CONN_4, P3 CONN_4, P4 CONN_4, P5 CONN_4, P6 CONN_4, P7 CONN_4, P8 CONN_4, P9 CONN_4, U1 A4982SLPTR, U10 USB_3.0_Receptacle, U11 KSZ8051RNL, U12 ATSAM3X8E, U13 USB_3.0_Receptacle_4, U14 USB_3.0_Receptacle_4, U15 USB_3.0_Receptacle_4, U16 USB_3.0_Receptacle_4, U17 USB_3.0_Receptacle_4, U18 USB_3.0_Receptacle_3, U19 USB_3.0_Receptacle_2, U2 A4982SLPTR, U20 USB_3.0_Receptacle_2, U21 USB_3.0_Receptacle_3, U3 A4982SLPTR, U4 A4982SLPTR, U5 A4982SLPTR, U6 MCP44X1, U7 TC2117-3.3VDBTR, U8 A4403, U9 USB_3.0_Receptacle, X1 CRYSTAL_4PIN, X2 CRYSTAL_4PIN

Commit message: More routing, even under crystals.
Parts:
- J10, J11: value GND V_IN -> GND V_IN
- moved R74 14.7 mm to (60.0, 73.8), turned to 0 degrees
- moved C61 14.2 mm to (60.1, 70.5), turned to 180 degrees
- moved C60 12.9 mm to (60.1, 68.8), turned to 180 degrees
- moved R73 9.64 mm to (60.0, 72.1), turned to 180 degrees
- moved R105 6.60 mm to (109.1, 57.6), turned to 0 degrees
- moved R102 5.85 mm to (103.2, 57.6)
- moved R106 4.19 mm to (97.9, 72.8)
- moved R108 3.91 mm to (94.7, 73.7)
- moved C53 2.40 mm to (72.6, 70.7)
- moved R53 2.40 mm to (86.0, 70.7)
- moved R56 2.40 mm to (77.5, 70.7)
- moved R57 2.40 mm to (79.1, 70.7)
- moved R60 2.40 mm to (84.3, 70.7)
- moved J20 2.40 mm to (79.6, 56.3)
- moved R52 2.40 mm to (80.7, 70.7)
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Connections:
- net PC4_PWML1 renamed FAN1_PWM
- J6 pad 21: LED0_B_PWM -> Net-(J6-Pad21)
- J6 pad 22: PC22_PWML5 -> Net-(J6-Pad22)
- J6 pad 23: LED0_G_PWM -> Net-(J6-Pad23)
- J6 pad 24: LED1_G_PWM -> Net-(J6-Pad24)
- J6 pad 49: PC18_PWMH6 -> Net-(J6-Pad49)
- J6 pad 50: PC19_PWMH5 -> Net-(J6-Pad50)
- R86 pad 1: LED0_G_PWM -> PC21_PWML4
- R87 pad 1: LED1_G_PWM -> PC20_PWMH4
- R94 pad 1: LED0_B_PWM -> PC23_PWML6
- R95 pad 1: PC18_PWMH6 -> LED1_B_PWM
- TR10 pad G: LED0_B_PWM -> PC23_PWML6
- TR11 pad G: PC18_PWMH6 -> LED1_B_PWM
- TR6 pad G: LED0_G_PWM -> PC21_PWML4
- TR7 pad G: LED1_G_PWM -> PC20_PWMH4
- U12 pad 100: PC18_PWMH6 -> LED1_B_PWM
- U12 pad 131: LED1_G_PWM -> PC20_PWMH4
- U12 pad 132: LED0_G_PWM -> PC21_PWML4
- U12 pad 134: LED0_B_PWM -> PC23_PWML6
Routing:
- net (no net): track 0.00 -> 3402.0 mm
- net RESET: track 0.00 -> 147.1 mm, vias 0 -> 1
- net Net-(J21-Pad6): track 0.00 -> 143.8 mm, vias 0 -> 2
- net Net-(J21-Pad11): track 0.00 -> 142.3 mm, vias 0 -> 1
- net Net-(J21-Pad3): track 0.00 -> 135.6 mm, vias 0 -> 2
- net Net-(J21-Pad2): track 0.00 -> 133.3 mm, vias 0 -> 2
- net Net-(J21-Pad1): track 0.00 -> 128.1 mm, vias 0 -> 2
- net Net-(J21-Pad10): track 0.00 -> 127.7 mm, vias 0 -> 4
- net AD12: track 0.00 -> 123.0 mm, vias 0 -> 6
- net PC10: track 0.00 -> 104.7 mm, vias 0 -> 1
- net +3.3V: track 137.5 -> 237.5 mm, vias 0 -> 9
- net E1_THERMISTOR: track 13.2 -> 91.9 mm, vias 0 -> 2
- net E0_THERMISTOR: track 76.1 -> 151.5 mm, vias 2 -> 4
- net MCDA2: track 3.14 -> 76.0 mm, vias 0 -> 4
- net BED_THERMISTOR: track 95.3 -> 168.1 mm, vias 2 -> 4
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