File: Duet-master/Duet0.8.5/Processor.sch (KiCad schematic (older format))
At the start: 43 parts, among them J23 JTAG, J24 GND, U12 ATSAM3X8E, X2 CRYSTAL_4PIN

Commit message: PCB layout of components started
Experienced advice welcome.
Parts:
- C69: footprint (none) -> Melter_Connections:10mf_capacitor
- C70, C72, C74, C75, C78, C79, C81, C82, C84, C86, C87, C89, C90, C91: footprint (none) -> Melter_Connections:0mf1_capacitor
- C71, C73, C83, C85: footprint (none) -> Melter_Connections:4uf7_capacitor
- C76, C77, C80: footprint (none) -> Melter_Connections:10pf_capacitor
- C88: footprint (none) -> Melter_Connections:10nf_capacitor
- C92: footprint (none) -> Melter_Connections:0mf01_Capacitor
- J23: footprint (none) -> Melter_Connections:PIN_ARRAY_5x2
- J24: footprint (none) -> Melter_Connections:GND_TP
- L3, L4, L5, L6, L7: footprint (none) -> Melter_Connections:100Mhz_R_0603
- R102, R104, R105: footprint (none) -> Melter_Connections:100k_R_0603
- R103: footprint (none) -> Melter_Connections:6k8_R_0603
- R106, R107, R108, R109: footprint (none) -> Melter_Connections:10k_R_0603
- S1, S2: footprint (none) -> Melter_Connections:SW_SIDE_1
- U12: footprint LQFP100 -> Melter_Connections:LQFP144
- X2: footprint (none) -> Melter_Connections:Xtal_5x3.2

Commit message: More routing
Connections:
- net PC4_PWML1 renamed FAN1_PWM
- net PC7_PWMH2 renamed E2_STOP
Changed lines of the file:
@@
 PC20_PWMH4
 Text GLabel 13750 8000 2    50   BiDi ~ 0
-PC4_PWML1
+FAN1_PWM
 Text GLabel 13750 9800 2    50   BiDi ~ 0
 PC19_PWMH5
@@
 E1_PWM
 Text GLabel 10350 9650 0    50   BiDi ~ 0
-PC7_PWMH2
+E2_STOP
 Text Label 10650 2900 0    60   ~ 0
 VDDIO
